File: Pcb/SensorToAmbient/SensorToAmbient.sch (KiCad schematic (older format))
At the start: 14 parts, among them J1 Conn_01x04, J2 Conn_01x04, J3 Conn_01x04, J4 Conn_01x06, J5 Conn_01x02, J6 Conn_01x06, J7 Conn_01x04, J8 Conn_01x04, J9 Conn_01x04

Commit message: Complete of footprint layout before first wiring work
Parts:
- J7: renamed from J5; footprint Connectors_JST:JST_XH_B02B-XH-A_02x2.50mm_Straight -> Connectors_JST:JST_XH_S02B-XH-A_02x2.50mm_Angled
- J8: renamed from J4; footprint Connectors_JST:JST_XH_B06B-XH-A_06x2.50mm_Straight -> Connectors_JST:JST_XH_S06B-XH-A_06x2.50mm_Angled
- J9: renamed from J6; footprint Connectors_JST:JST_XH_B06B-XH-A_06x2.50mm_Straight -> Connectors_JST:JST_XH_S06B-XH-A_06x2.50mm_Angled
- renumbered J8 to J4, J7 to J5, J9 to J6
Changed lines of the file:
@@
 $EndComp
 $Comp
-L SensorToAmbient-rescue:Conn_01x04-Connector_Grove J9
+L SensorToAmbient-rescue:Conn_01x04-Connector_Grove J6
 U 1 1 5BE0F456
 P 5100 2400
-F 0 "J9" H 5020 2717 50  0000 C CNN
+F 0 "J6" H 5020 2717 50  0000 C CNN
 F 1 "Conn_01x04" H 5020 2626 50  0000 C CNN
 F 2 "SensorToAmbient:Grove_2mm_4pin_angle" H 5100 2400 50  0001 C CNN
@@
 $EndComp
 $Comp
-L SensorToAmbient-rescue:Conn_01x04-Connector_Grove J8
+L SensorToAmbient-rescue:Conn_01x04-Connector_Grove J4
 U 1 1 5BE0F523
 P 5050 5100
-F 0 "J8" H 4970 5417 50  0000 C CNN
+F 0 "J4" H 4970 5417 50  0000 C CNN
 F 1 "Conn_01x04" H 4970 5326 50  0000 C CNN
 F 2 "SensorToAmbient:Grove_2mm_4pin_angle" H 5050 5100 50  0001 C CNN
@@
 $EndComp
 $Comp
-L SensorToAmbient-rescue:Conn_01x06-Connector_Generic J4
+L SensorToAmbient-rescue:Conn_01x06-Connector_Generic J8
 U 1 1 5BE0FB43
 P 2200 650
-F 0 "J4" V 2166 262 50  0000 R CNN
+F 0 "J8" V 2166 262 50  0000 R CNN
 F 1 "Conn_01x06" V 2075 262 50  0000 R CNN
-F 2 "Connectors_JST:JST_XH_B06B-XH-A_06x2.50mm_Straight" H 2200 650 50  0001 C CNN
+F 2 "Connectors_JST:JST_XH_S06B-XH-A_06x2.50mm_Angled" H 2200 650 50  0001 C CNN
 F 3 "~" H 2200 650 50  0001 C CNN
 	1    2200 650
@@
 $EndComp
 $Comp
-L SensorToAmbient-rescue:Conn_01x06-Connector_Generic J6
+L SensorToAmbient-rescue:Conn_01x06-Connector_Generic J9
 U 1 1 5BE0FBD1
 P 4000 650
-F 0 "J6" V 3966 262 50  0000 R CNN
+F 0 "J9" V 3966 262 50  0000 R CNN
 F 1 "Conn_01x06" V 3875 262 50  0000 R CNN
-F 2 "Connectors_JST:JST_XH_B06B-XH-A_06x2.50mm_Straight" H 4000 650 50  0001 C CNN
+F 2 "Connectors_JST:JST_XH_S06B-XH-A_06x2.50mm_Angled" H 4000 650 50  0001 C CNN
 F 3 "~" H 4000 650 50  0001 C CNN
 	1    4000 650
@@
 $EndComp
 $Comp
-L SensorToAmbient-rescue:Conn_01x02-Connector_Generic J5
+L SensorToAmbient-rescue:Conn_01x02-Connector_Generic J7
 U 1 1 5BE0FD4D
 P 3950 5900
-F 0 "J5" V 3823 5980 50  0000 L CNN
+F 0 "J7" V 3823 5980 50  0000 L CNN
 F 1 "Conn_01x02" V 3914 5980 50  0000 L CNN
-F 2 "Connectors_JST:JST_XH_B02B-XH-A_02x2.50mm_Straight" H 3950 5900 50  0001 C CNN
+F 2 "Connectors_JST:JST_XH_S02B-XH-A_02x2.50mm_Angled" H 3950 5900 50  0001 C CNN
 F 3 "~" H 3950 5900 50  0001 C CNN
 	1    3950 5900
@@
 	4800 3150 4800 3600
 $Comp
-L SensorToAmbient-rescue:Conn_01x04-Connector_I2C J7
+L SensorToAmbient-rescue:Conn_01x04-Connector_I2C J5
 U 1 1 5BE0F4CE
 P 5050 3600
-F 0 "J7" H 4970 3917 50  0000 C CNN
+F 0 "J5" H 4970 3917 50  0000 C CNN
 F 1 "Conn_01x04" H 4970 3826 50  0000 C CNN
 F 2 "SensorToAmbient:Grove_2mm_4pin_angle" H 5050 3600 50  0001 C CNN

Commit message: Commit intermediate (before revice part layout for wiring)
Connections:
- net labels added: PWR_BAT
Changed lines of the file:
@@
 	1    0    0    -1
 $EndComp
+Text Label 3850 5450 1    50   ~ 0
+PWR_BAT
 $EndSCHEMATC

Commit message: Commit intermediate (Revice schematic for pcb wiring)
Parts:
- J1, J2, J3, J4, J5, J6: footprint SensorToAmbient:Grove_2mm_4pin_angle -> SensorToAmbient:Grove_2mm_4pin_angle2
Connections:
- wire segments 119 -> 107
- no-connect marks 7 -> 16
Other:
- moved on the sheet: 3SB1, RTC1

Commit message: Commit intermediate (Remaining wire is only one GND)
Parts:
- J5: footprint SensorToAmbient:Grove_2mm_4pin_angle2 -> Connectors_JST:JST_XH_S04B-XH-A_04x2.50mm_Angled
Connections:
- wire segments 107 -> 110
Changed lines of the file:
@@
 L SensorToAmbient-rescue:Conn_01x02-Connector_Generic J7
 U 1 1 5BE0FD4D
-P 3950 5900
-F 0 "J7" V 3823 5980 50  0000 L CNN
-F 1 "Conn_01x02" V 3914 5980 50  0000 L CNN
-F 2 "Connectors_JST:JST_XH_S02B-XH-A_02x2.50mm_Angled" H 3950 5900 50  0001 C CNN
-F 3 "~" H 3950 5900 50  0001 C CNN
-	1    3950 5900
-	0    1    1    0
+P 3850 5900
+F 0 "J7" V 3723 5980 50  0000 L CNN
+F 1 "Conn_01x02" V 3814 5980 50  0000 L CNN
+F 2 "Connectors_JST:JST_XH_S02B-XH-A_02x2.50mm_Angled" H 3850 5900 50  0001 C CNN
+F 3 "~" H 3850 5900 50  0001 C CNN
+	1    3850 5900
+	0    -1   1    0
 $EndComp
 $Comp
@@
 L SensorToAmbient-rescue:Conn_01x04-Connector_I2C J5
 U 1 1 5BE0F4CE
-P 5050 3600
-F 0 "J5" H 4970 3917 50  0000 C CNN
-F 1 "Conn_01x04" H 4970 3826 50  0000 C CNN
-F 2 "SensorToAmbient:Grove_2mm_4pin_angle2" H 5050 3600 50  0001 C CNN
-F 3 "~" H 5050 3600 50  0001 C CNN
-	1    5050 3600
-	1    0    0    -1
+P 5050 3700
+F 0 "J5" H 4970 4017 50  0000 C CNN
+F 1 "Conn_01x04" H 4970 3926 50  0000 C CNN
+F 2 "Connectors_JST:JST_XH_S04B-XH-A_04x2.50mm_Angled" H 5050 3700 50  0001 C CNN
+F 3 "~" H 5050 3700 50  0001 C CNN
+	1    5050 3700
+	1    0    0    1
 $EndComp
 NoConn ~ 2900 5200
@@
 	1    0    0    -1
 $EndComp
-Wire Wire Line
-	4600 5550 4600 5900
 Connection ~ 4600 5550
 Wire Wire Line
@@
 	1    0    0    -1
 $EndComp
-Wire Wire Line
-	2100 4950 2100 5300
 Connection ~ 2100 4950
 Wire Wire Line
@@
 	2000 1100 2000 3850
 Wire Wire Line
-	5200 3800 4850 3800
-Wire Wire Line
 	2900 4900 3850 4900
 Wire Wire Line
@@
 Connection ~ 4750 2450
 Wire Wire Line
-	4750 2450 4750 3500
-Wire Wire Line
-	4850 3500 4750 3500
-Wire Wire Line
-	4850 3600 4650 3600
-Wire Wire Line
-	4650 2550 4650 3600
+	4650 2550 4650 3500
 Wire Wire Line
 	5250 6200 5250 3700
-Wire Wire Line
-	5250 3700 4850 3700
 Wire Wire Line
 	3300 6200 5250 6200
@@
 Connection ~ 4100 1100
 Wire Wire Line
-	4300 2750 4300 3700
-Wire Wire Line
-	4300 3700 4850 3700
-Connection ~ 4850 3700
-Wire Wire Line
 	3400 2750 3400 3800
-Wire Wire Line
-	3400 3800 4850 3800
-Connection ~ 4850 3800
-Wire Wire Line
-	2100 5300 2700 5300
-Connection ~ 2100 5300
-Wire Wire Line
-	2100 5300 2100 5950
 Connection ~ 2900 5300
 NoConn ~ 3050 2700
@@
 Wire Wire Line
 	2700 2300 2700 5300
-Connection ~ 2700 5300
 Wire Wire Line
 	2700 5300 2900 5300
@@
 Wire Wire Line
 	3400 1800 3400 2450
+Wire Wire Line
+	4650 3500 4750 3500
+Wire Wire Line
+	4850 3600 4750 3600
+Wire Wire Line
+	4750 3500 4850 3500
+Wire Wire Line
+	4750 2450 4750 3600
+Wire Wire Line
+	3400 3800 4850 3800
+Connection ~ 4850 3800
+Wire Wire Line
+	4850 3800 5200 3800
+Wire Wire Line
+	5250 3700 4850 3700
+Wire Wire Line
+	4300 2750 4300 3150
+Wire Wire Line
+	4300 3150 3850 3150
+Wire Wire Line
+	3850 3150 3850 4700
+Connection ~ 3850 4700
+Wire Wire Line
+	2100 4950 2100 5950
+Wire Wire Line
+	4300 900  5300 900
+Wire Wire Line
+	5300 900  5300 5550
+Connection ~ 4300 900
+Text Label 4700 5550 2    50   ~ 0
+GND
+Wire Wire Line
+	4600 5550 4600 5900
+Wire Wire Line
+	5300 5550 5200 5550
+Connection ~ 5200 5550
 $EndSCHEMATC

Commit message: First comple of wiring
Connections:
- wire segments 110 -> 114
- no-connect marks 16 -> 15
Changed lines of the file:
@@
 Connection ~ 2200 900
 Wire Wire Line
-	2200 900  2200 5050
+	2200 900  2200 2900
 Wire Wire Line
 	2100 1000 4200 1000
@@
 	3800 1300 3800 850
 Wire Wire Line
-	1800 2400 2250 2400
-Wire Wire Line
-	1800 850  1800 2400
-Wire Wire Line
-	1500 2450 2250 2450
-Wire Wire Line
-	2250 2450 2250 2500
-Wire Wire Line
 	3900 850  3900 1900
-Wire Wire Line
-	3900 1900 3200 1900
-Wire Wire Line
-	3200 1900 3200 2500
-Wire Wire Line
-	3200 2500 3050 2500
-Wire Wire Line
-	2250 2300 2250 2100
-Wire Wire Line
-	2250 2100 2650 2100
 Wire Wire Line
 	2650 2100 2650 4300
@@
 Wire Wire Line
 	1500 5250 2000 5250
-Wire Wire Line
-	3050 2400 3150 2400
-Wire Wire Line
-	3150 2100 2650 2100
-Connection ~ 2650 2100
 Wire Wire Line
 	4650 2200 4900 2200
@@
 Wire Wire Line
 	4500 4550 3200 4550
-Wire Wire Line
-	3200 4550 3200 2600
-Wire Wire Line
-	3200 2600 3050 2600
 Connection ~ 2000 1100
 Wire Wire Line
@@
 Wire Wire Line
 	3400 2750 3400 3800
-Connection ~ 2900 5300
 NoConn ~ 3050 2700
 NoConn ~ 3050 2800
 NoConn ~ 3050 2900
-NoConn ~ 2250 2900
-NoConn ~ 2250 2800
-NoConn ~ 2250 2700
-NoConn ~ 2250 2600
-Wire Wire Line
-	3150 2400 3150 2100
-Wire Wire Line
-	3050 2300 2700 2300
-Wire Wire Line
-	2700 2300 2700 5300
-Wire Wire Line
-	2700 5300 2900 5300
 Wire Wire Line
 	1500 2550 1600 2550
@@
 	5300 5550 5200 5550
 Connection ~ 5200 5550
+Wire Wire Line
+	2250 2900 2200 2900
+Connection ~ 2200 2900
+Wire Wire Line
+	2200 2900 2200 5050
+Wire Wire Line
+	1500 2450 1750 2450
+Wire Wire Line
+	1750 2450 1750 2800
+Wire Wire Line
+	1750 2800 2250 2800
+Wire Wire Line
+	1800 2700 2250 2700
+Wire Wire Line
+	1800 850  1800 2700
+Wire Wire Line
+	2150 2100 2150 2300
+Wire Wire Line
+	2150 2600 2250 2600
+Wire Wire Line
+	2150 2100 2650 2100
+Wire Wire Line
+	2050 1900 2050 2400
+Wire Wire Line
+	2050 2400 2250 2400
+Wire Wire Line
+	2050 1900 3900 1900
+Wire Wire Line
+	2250 2300 2150 2300
+Connection ~ 2150 2300
+Wire Wire Line
+	2150 2300 2150 2600
+Wire Wire Line
+	3200 2450 2250 2450
+Wire Wire Line
+	2250 2450 2250 2500
+Wire Wire Line
+	3200 2450 3200 4550
+NoConn ~ 3050 2400
+NoConn ~ 3050 2500
+NoConn ~ 3050 2600
+Wire Wire Line
+	3050 2300 3300 2300
+Wire Wire Line
+	3300 2300 3300 2750
+Wire Wire Line
+	3300 2750 3400 2750
+Connection ~ 3400 2750
 $EndSCHEMATC

Commit message: Fix DRC errors
Connections:
- wire segments 114 -> 110
- no-connect marks 15 -> 17
Changed lines of the file:
@@
 Wire Wire Line
 	2100 850  2100 1000
-Text Label 2200 1700 1    50   ~ 0
-PWR3.3V
 Wire Wire Line
 	2200 850  2200 900
@@
 NoConn ~ 3050 2900
 Wire Wire Line
-	1500 2550 1600 2550
-Wire Wire Line
-	1600 2550 1600 1800
-Wire Wire Line
-	1600 1800 3400 1800
-Wire Wire Line
-	3400 1800 3400 2450
-Wire Wire Line
 	4650 3500 4750 3500
 Wire Wire Line
@@
 	2100 4950 2100 5950
 Wire Wire Line
-	4300 900  5300 900
-Wire Wire Line
-	5300 900  5300 5550
-Connection ~ 4300 900
+	5300 1000 5300 5550
 Text Label 4700 5550 2    50   ~ 0
 GND
@@
 	3300 2750 3400 2750
 Connection ~ 3400 2750
+Text Label 2200 1700 1    50   ~ 0
+PWR3.3V
+Wire Wire Line
+	5300 1000 4200 1000
+Connection ~ 4200 1000
+NoConn ~ 1500 2550
+NoConn ~ 3400 2450
 $EndSCHEMATC

Commit message: Make ground plane
Connections:
- wire segments 110 -> 111
Changed lines of the file:
@@
 	3300 6200 5250 6200
-Wire Wire Line
-	3950 5850 3950 6050
-Wire Wire Line
-	3950 6050 3400 6050
 Wire Wire Line
 	3400 6050 3400 5300
@@
 NoConn ~ 1500 2550
 NoConn ~ 3400 2450
+Wire Wire Line
+	4050 6050 4050 5700
+Wire Wire Line
+	4050 5700 3950 5700
+Wire Wire Line
+	3400 6050 4050 6050
+Connection ~ 3950 5700
 $EndSCHEMATC

Commit message: Commit intermediate (Add items for power controll)
Parts:
- added D?: DIODE, symbol pspice:DIODE
- added R?: R, symbol device:R
- added SW?: SW_Push, symbol Switch:SW_Push
Connections:
- wire segments 111 -> 127
- no-connect marks 17 -> 14
