File: Pcb/SensorToAmbient/SensorToAmbient.kicad_pcb (KiCad board)
At the start: 2 copper layers, 48.1 x 77.7 mm, 30 parts, among them J1 Conn_01x04, J2 Conn_01x04, J3 Conn_01x04, J4 Conn_01x04, J5 Conn_01x04, J6 Conn_01x04, J7 Conn_01x02, J8 Conn_01x06, J9 Conn_01x06, SW1 SW_Push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

Commit message: Complete running with only battery
Parts:
- removed R7: 47K, Resistors_SMD:R_0805_HandSoldering
- R3: value 47K -> 100K
- R6: value 47K -> 10K
- R8, R9: value 4.7K -> 10K
- moved D1 4.93 mm to (44.7, 78.0)
Connections:
- D1 pad 2: Net-(D1-Pad2) -> /PWR_BAT
Routing:
- net Net-(D1-Pad2): track 3.40 -> 0.00 mm
- net Net-(D1-Pad1): track 6.72 -> 9.00 mm
- net GND: track 209.6 -> 208.2 mm
Changed lines of the file:
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@@
     (thickness 1.6)
     (drawings 10)
-    (tracks 243)
+    (tracks 240)
     (zones 0)
-    (modules 30)
-    (nets 37)
+    (modules 29)
+    (nets 36)
   )
   (page A4)
@@
   (net 34 /PWR3.3V_Sensors)
   (net 35 "Net-(D2-Pad1)")
-  (net 36 "Net-(D1-Pad2)")
   (net_class Default "これはデフォルトのネット クラスです。"
     (clearance 0.2)
@@
     (add_net "Net-(3SB1-Pad9)")
     (add_net "Net-(D1-Pad1)")
-    (add_net "Net-(D1-Pad2)")
     (add_net "Net-(D2-Pad1)")
     (add_net "Net-(DCDC1-Pad4)")
@@
   )
   (module Diodes_SMD:D_SOD-323_HandSoldering (layer F.Cu)
-    (at 40 76.5)
+    (at 44.704 77.978)
     (descr SOD-323)
     (tags SOD-323)
@@
       (net 28 "Net-(D1-Pad1)"))
     (pad 2 smd rect (at 1.25 0) (size 1 1) (layers F.Cu F.Paste F.Mask)
-      (net 36 "Net-(D1-Pad2)"))
+      (net 15 /PWR_BAT))
     (model ${KISYS3DMOD}/Diodes_SMD.3dshapes/D_SOD-323.wrl
       (at (xyz 0 0 0))
@@
       (effects (font (size 1 1) (thickness 0.15)))
     )
-    (fp_text value 4.7K (at 0 1.75) (layer F.Fab)
+    (fp_text value 10K (at 0 1.75) (layer F.Fab)
       (effects (font (size 1 1) (thickness 0.15)))
     )
@@
       (effects (font (size 1 1) (thickness 0.15)))
     )
-    (fp_text value 47K (at 0 1.75 90) (layer F.Fab)
+    (fp_text value 10K (at 0 1.75 90) (layer F.Fab)
       (effects (font (size 1 1) (thickness 0.15)))
     )
@@
   )
   (module Resistors_SMD:R_0805_HandSoldering (layer F.Cu)
-    (at 46 76.5 180)
-    (descr "Resistor SMD 0805, hand soldering")
-    (tags "resistor 0805")
-    (attr smd)
-    (fp_text reference R7 (at 0 -1.7 180) (layer F.SilkS)
-      (effects (font (size 1 1) (thickness 0.15)))
-    )
-    (fp_text value 47K (at 0 1.75 180) (layer F.Fab)
-      (effects (font (size 1 1) (thickness 0.15)))
-    )
-    (fp_line (start 2.35 0.9) (end -2.35 0.9) (layer F.CrtYd) (width 0.05))
-    (fp_line (start 2.35 0.9) (end 2.35 -0.9) (layer F.CrtYd) (width 0.05))
-    (fp_line (start -2.35 -0.9) (end -2.35 0.9) (layer F.CrtYd) (width 0.05))
-    (fp_line (start -2.35 -0.9) (end 2.35 -0.9) (layer F.CrtYd) (width 0.05))
-    (fp_line (start -0.6 -0.88) (end 0.6 -0.88) (layer F.SilkS) (width 0.12))
-    (fp_line (start 0.6 0.88) (end -0.6 0.88) (layer F.SilkS) (width 0.12))
-    (fp_line (start -1 -0.62) (end 1 -0.62) (layer F.Fab) (width 0.1))
-    (fp_line (start 1 -0.62) (end 1 0.62) (layer F.Fab) (width 0.1))
-    (fp_line (start 1 0.62) (end -1 0.62) (layer F.Fab) (width 0.1))
-    (fp_line (start -1 0.62) (end -1 -0.62) (layer F.Fab) (width 0.1))
-    (fp_text user %R (at 0 0 180) (layer F.Fab)
-      (effects (font (size 0.5 0.5) (thickness 0.075)))
-    )
-    (pad 2 smd rect (at 1.35 0 180) (size 1.5 1.3) (layers F.Cu F.Paste F.Mask)
-      (net 36 "Net-(D1-Pad2)"))
-    (pad 1 smd rect (at -1.35 0 180) (size 1.5 1.3) (layers F.Cu F.Paste F.Mask)
-      (net 15 /PWR_BAT))
-    (model ${KISYS3DMOD}/Resistors_SMD.3dshapes/R_0805.wrl
-      (at (xyz 0 0 0))
-      (scale (xyz 1 1 1))
-      (rotate (xyz 0 0 0))
-    )
-  )
-  (module Resistors_SMD:R_0805_HandSoldering (layer F.Cu)
     (at 62.15 32.25)
     (descr "Resistor SMD 0805, hand soldering")
@@
       (effects (font (size 1 1) (thickness 0.15)))
     )
-    (fp_text value 4.7K (at 0 1.75) (layer F.Fab)
+    (fp_text value 10K (at 0 1.75) (layer F.Fab)
       (effects (font (size 1 1) (thickness 0.15)))
     )
@@
       (effects (font (size 1 1) (thickness 0.15)))
     )
-    (fp_text value 47K (at 0 1.75 90) (layer F.Fab)
+    (fp_text value 100K (at 0 1.75 90) (layer F.Fab)
       (effects (font (size 1 1) (thickness 0.15)))
     )
@@
   (segment (start 46.958 83.054) (end 45.907999 84.104001) (width 0.5) (layer F.Cu) (net 4) (status 10))
   (segment (start 46.958 82.804) (end 46.958 83.054) (width 0.5) (layer F.Cu) (net 4) (status 30))
-  (segment (start 43.75 81.751998) (end 43.75 84.104001) (width 0.5) (layer F.Cu) (net 4))
-  (segment (start 45.850001 79.651997) (end 43.75 81.751998) (width 0.5) (layer F.Cu) (net 4))
-  (segment (start 46.239999 75.399999) (end 45.850001 75.789997) (width 0.5) (layer F.Cu) (net 4))
-  (segment (start 45.850001 75.789997) (end 45.850001 79.651997) (width 0.5) (layer F.Cu) (net 4))
-  (segment (start 54.505499 75.399999) (end 46.239999 75.399999) (width 0.5) (layer F.Cu) (net 4))
-  (segment (start 55.805 76.6995) (end 54.505499 75.399999) (width 0.5) (layer F.Cu) (net 4) (status 10))
   (segment (start 43.75 84.104001) (end 33.775999 84.104001) (width 0.5) (layer F.Cu) (net 4))
   (segment (start 45.907999 84.104001) (end 43.75 84.104001) (width 0.5) (layer F.Cu) (net 4))
+  (segment (start 43.75 81.751998) (end 43.75 84.104001) (width 0.5) (layer F.Cu) (net 4))
+  (segment (start 44.404001 81.097997) (end 43.75 81.751998) (width 0.5) (layer F.Cu) (net 4))
+  (segment (start 44.404001 77.717997) (end 44.404001 81.097997) (width 0.5) (layer F.Cu) (net 4))
+  (segment (start 45.422498 76.6995) (end 44.404001 77.717997) (width 0.5) (layer F.Cu) (net 4))
+  (segment (start 55.805 76.6995) (end 45.422498 76.6995) (width 0.5) (layer F.Cu) (net 4))
   (segment (start 62.15 70.29) (end 62.15 66.003498) (width 0.25) (layer B.Cu) (net 5) (status 10))
   (segment (start 38.295021 44.125021) (end 36.27 42.1) (width 0.25) (layer B.Cu) (net 5) (status 20))
@@
   (segment (start 44.958 82.554) (end 49.534 77.978) (width 0.5) (layer F.Cu) (net 15) (status 10))
   (segment (start 44.958 82.804) (end 44.958 82.554) (width 0.5) (layer F.Cu) (net 15) (status 30))
-  (segment (start 47.678 77.978) (end 49.534 77.978) (width 0.5) (layer F.Cu) (net 15))
-  (segment (start 47.35 77.65) (end 47.678 77.978) (width 0.5) (layer F.Cu) (net 15))
-  (segment (start 47.35 76.5) (end 47.35 77.65) (width 0.5) (layer F.Cu) (net 15) (status 10))
   (segment (start 54.531738 69.6) (end 54.592999 69.661261) (width 0.5) (layer F.Cu) (net 15))
   (segment (start 51 69.6) (end 54.531738 69.6) (width 0.5) (layer F.Cu) (net 15) (status 10))
@@
   (segment (start 57.450001 43.640001) (end 57.450001 59.688499) (width 0.5) (layer F.Cu) (net 15))
   (segment (start 56.2 42.39) (end 57.450001 43.640001) (width 0.5) (layer F.Cu) (net 15) (status 10))
+  (segment (start 46.954 77.978) (end 49.534 77.978) (width 0.5) (layer F.Cu) (net 15))
+  (segment (start 45.954 77.978) (end 46.954 77.978) (width 0.5) (layer F.Cu) (net 15))
   (segment (start 63.300001 51.799999) (end 61.24 53.86) (width 0.25) (layer B.Cu) (net 16) (status 20))
   (segment (start 63.300001 41.240001) (end 63.300001 51.799999) (width 0.25) (layer B.Cu) (net 16))
@@
   (segment (start 53.16 19.55) (end 51.959999 20.750001) (width 0.25) (layer B.Cu) (net 26) (status 10))
   (segment (start 36.576 81.764) (end 36.536 81.804) (width 0.25) (layer B.Cu) (net 28) (status 30))
-  (segment (start 38 76.5) (end 38.75 76.5) (width 0.25) (layer F.Cu) (net 28) (status 20))
-  (segment (start 36.536 77.964) (end 38 76.5) (width 0.25) (layer F.Cu) (net 28))
-  (segment (start 36.536 81.804) (end 36.536 77.964) (width 0.25) (layer F.Cu) (net 28) (status 10))
+  (segment (start 43.454 78.728) (end 43.454 77.978) (width 0.25) (layer F.Cu) (net 28))
+  (segment (start 40.378 81.804) (end 43.454 78.728) (width 0.25) (layer F.Cu) (net 28))
+  (segment (start 36.536 81.804) (end 40.378 81.804) (width 0.25) (layer F.Cu) (net 28))
   (segment (start 45.015001 48.305001) (end 45.015001 60.984999) (width 0.25) (layer F.Cu) (net 29))
   (segment (start 43.89 47.18) (end 45.015001 48.305001) (width 0.25) (layer F.Cu) (net 29) (status 10))
@@
   (segment (start 44.25 69.6) (end 45.15 69.6) (width 0.25) (layer F.Cu) (net 35) (status 10))
   (segment (start 45.15 69.6) (end 47.1695 71.6195) (width 0.25) (layer F.Cu) (net 35))
-  (segment (start 41.25 76.5) (end 44.65 76.5) (width 0.25) (layer F.Cu) (net 36) (status 30))
   (zone (net 4) (net_name GND) (layer F.Cu) (hatch edge 0.508)
     (connect_pads (clearance 0.508))
@@
     (polygon
       (pts
-        (xy 21 7) (xy 73 7) (xy 73 90.5) (xy 20.75 90.5) (xy 20.25 90)
+        (xy 20.32 7.366) (xy 72.644 7.366) (xy 72.644 90.17) (xy 20.828 90.17)
       )
     )
